File: ExtraUserPort.sch (KiCad schematic (older format))
At the start: 28 parts, among them CN1 EXPANSION_PORT, CN2 ALMOST_USERPORT

Commit message: Assign footprints
Parts:
- C2, C4: renamed from C?; footprint (none) -> Capacitor_THT:C_Disc_D7.0mm_W2.5mm_P5.00mm
- C5, C6, C7, C8, C9: renamed from C?; footprint (none) -> Capacitor_THT:CP_Radial_D5.0mm_P2.00mm
- CN1: footprint MODULE -> ExtraUserPort:C16_Cart_Conn
- CN2: footprint MODULE -> ExtraUserPort:24Pin_Edge
- CN3: renamed from CN?; footprint Plus4Serial:DB_9M -> ExtraUserPort:DB_9M
- J1: renamed from J?; footprint (none) -> Connector_PinHeader_2.54mm:PinHeader_1x01_P2.54mm_Vertical
- R1, R2: renamed from R?; footprint (none) -> Resistor_THT:R_Axial_DIN0207_L6.3mm_D2.5mm_P10.16mm_Horizontal
- U2: renamed from U?; footprint MODULE -> Package_DIP:DIP-20_W7.62mm_Socket_LongPads
- U3: renamed from U?; footprint MODULE -> Package_DIP:DIP-28_W15.24mm_Socket_LongPads
- U4: renamed from U?; footprint (none) -> Package_DIP:DIP-14_W7.62mm_Socket_LongPads
- U5: renamed from U?; footprint MODULE -> Package_DIP:DIP-24_W7.62mm_Socket_LongPads
- Y1: renamed from Y?; footprint (none) -> Crystal:Crystal_HC49-U_Vertical
- gave numbers to parts that had none: 3
Connections:
- net labels removed: rxc

Commit message: Fix some warnings
Connections:
- net labels removed: dcd
- wire segments 257 -> 259
- no-connect marks 20 -> 26
Other:
- note added: "MMMH... MAYBE RI COULD BE\nCONNECTED TO A DATA PIN\n(OR ~ATTN~?) THROUGH A DIODE?"
- note added: "THE W65C51S IS A DROP IN\nREPLACEMENT FOR THE ORIGINAL\nMOS6551.\n\nWHAT IS DIFFERENT IN THE W65C51N\nIS UNCLEAR TO ME!"
- note removed: "MMMH... MAYBE RI COULD BE\nCONNECTED TO A DATA PIN\n(OR ~ATTN?) THROUGH A DIODE?"
- moved on the sheet: C3, R1, R2, U3, Y1

Commit message: (Very) Rough routing done
Parts:
- added JP1: JMP_ACIA_ADDR, Connector_PinHeader_2.54mm:PinHeader_2x02_P2.54mm_Vertical, symbol Connector_Generic:Conn_02x02_Odd_Even
- added JP2: JMP_CTS_IN, Connector_PinHeader_2.54mm:PinHeader_1x03_P2.54mm_Vertical, symbol Connector:Conn_01x03_Male
- added JP3: JMP_CTS_ACIA, Connector_PinHeader_2.54mm:PinHeader_1x03_P2.54mm_Vertical, symbol Connector:Conn_01x03_Male
- J1: value ATTENTION -> ATTENTION_IN
- U3: value W65C51S -> MOS_6551_ACIA
Connections:
- net labels added: bit0, bit1, r_~w
- net labels removed: r_w~
- wire segments 259 -> 269
- no-connect marks 26 -> 25
Other:
- note added: "$FD60-FD63\n(CONFIGURABLE WITH J2)"
- note added: "+4 HAS NO DEDICATED ~CTS~ PIN.\nIT SEEMS THE SIGNAL WAS PLANNED\nTO BE CONNECTED TO D1, WHICH IS\nON PIN K ON THE USERPORT CONNECTOR,\nEXACTLY WHERE IT WOULD BE ON THE\nC64, THUS SOFTWARE SHOULD HAVE BEEN\nABLE TO POLL THAT PIN AND APPLY\nSOFTWARE FLOW CONTROL, I GUESS."
- note added: "IF AN ORIGINAL ACIA (MOS 6551)\nCANNOT BE OBTAINED, THE W65C51S\nIS A DROP-IN REPLACEMENT FOR IT\nTHAT IS STILL IN PRODUCTION.\n\nTHERE IS ALSO THE W65C51N, I'M\nNOT SURE WHAT DIFFERENCES IT\nHAS WRT THE -S MODEL THOUGH."
- note added: "MMMH... MAYBE RI COULD\nBE CONNECTED TO A DATA\nPIN SOMEHOW?"
- note added: "NO WAY WE\nCAN HAVE\n9VAC HERE!"
- note added: "SINCE WE ARE CONNECTED DIRECTLY\nTO THE RS-232 PORT, WITHOUT HAVING\nTO GO THROUGH THE USER PORT\nCONNECTOR, WE HAVE ~CTS~ AVAILABLE.\nLET'S CONNECT IT IN THE PROPER PLACE,\nBUT LET'S ALSO HAVE A JUMPER TO\nGROUND IT LIKE IN THE ORIGINAL +4\nCIRCUIT, JUST IN CASE."
- note added: "SINCE WE HAVE A MAX238 ONBOARD, IT WILL DRIVE THE SIGNALS\nTHAT ARE NORMALLY AN EXTERNAL INPUT THROUGH THIS PORT.\nIF ACCESS TO THOSE SIGNALS IS REQUIRED, THE MAX238 SHALL\nBE REMOVED FROM ITS SOCKET."
- note added: "WE PROVIDE A PIN\nFOR CONNECTION\nTO REAL ~ATTN~ LINE,\nJUST IN CASE"
- note removed: "$FD60-FD63 (CONFIGURABLE)"
- note removed: "+4 HAS NO DEDICATED ~CTS PIN. IT SEEMS THE SIGNAL WAS DESTINATED\nTO D1, WHICH IS ON PIN K, EXACTLY WHERE IT WOULD BE ON THE C64,\nTHUS SOFTWARE SHOULD POLL THAT PIN AND APPLY SOFTWARE FLOW\nCONTROL, I GUESS.\n\nBUT SINCE WE CAN BYPASS THE USERPORT CONNECTOR, WHY NOT CONNECT\n~CTS IN THE PROPER PLACE? ANY DRAWBACKS? MAYBE WE SHOULD\nINTRODUCE A JUMPER."
- note removed: "MMMH... MAYBE RI COULD BE\nCONNECTED TO A DATA PIN\n(OR ~ATTN~?) THROUGH A DIODE?"
- note removed: "NO WAY WE CAN\nHAVE 9VAC HERE!"
- note removed: "THE W65C51S IS A DROP IN\nREPLACEMENT FOR THE ORIGINAL\nMOS6551.\n\nWHAT IS DIFFERENT IN THE W65C51N\nIS UNCLEAR TO ME!"
- note removed: "WE PROVIDE A PIN\nFOR CONNECTION\nTO REAL ~ATTN\nLINE, JUST IN CASE"
- note removed: "WHAT TO DO\nWITH THESE???"
- moved on the sheet: C1, C2, C3, C4, C5, C6, C7, C8, C9, CN2, CN3, J1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

Commit message: Improve routing
Parts:
- removed C4: 100n, Capacitor_THT:C_Disc_D7.0mm_W2.5mm_P5.00mm, symbol Device:C
- removed U4: 74HCT04, Package_DIP:DIP-14_W7.62mm_Socket_LongPads, symbol 74xx:74HCT04
- added R3: 10k, Resistor_THT:R_Axial_DIN0207_L6.3mm_D2.5mm_P10.16mm_Horizontal, symbol Device:R
Connections:
- wire segments 269 -> 253
- no-connect marks 25 -> 21
Other:
- note added: "$FD60-FD63\n(CONFIGURABLE WITH JP1)"
- note removed: "$FD60-FD63\n(CONFIGURABLE WITH J2)"
- note removed: "SPARES"
- note removed: "WHY ARE SOME SIGNALS INVERTED???\n\nWHAT ABOUT ~CTS~???"
- moved on the sheet: C2, C3, JP3, R1, R2, U2B, U3, Y1

Commit message: Swap top/bottom pins of edge connector Sigh...
Other:
- note added: "BOTTOM"
- note added: "TOP"
Changed lines of the file:
@@
 Wire Bus Line
 	3630 2205 3630 3705
+Text Notes 13700 1545 0    50   ~ 0
+TOP
+Text Notes 14830 1545 0    50   ~ 0
+BOTTOM
 $EndSCHEMATC

Commit message: WIP
Parts:
- removed JP1: JMP_ACIA_ADDR, Connector_PinHeader_2.54mm:PinHeader_2x02_P2.54mm_Vertical, symbol Connector_Generic:Conn_02x02_Odd_Even
- removed U1: GAL16V8, Package_DIP:DIP-20_W7.62mm_Socket_LongPads, symbol Logic_Programmable:GAL16V8
- added JP1: JMP_ADDRESS, Connector_PinHeader_2.54mm:PinHeader_1x03_P2.54mm_Vertical, symbol Connector:Conn_01x03_Male
- added U1: GAL20V8, Package_DIP:DIP-24_W7.62mm_Socket_LongPads, symbol Logic_Programmable:PAL20L8
Connections:
- net +5V: now also JP1.3 (Pin_3), U1.24 (VCC)
- net GND: now also JP1.1 (Pin_1), U1.12 (GND)
- net a10: now also U1.6 (I6)
- net a11: now also U1.5 (I5)
- net a12: now also U1.4 (I4)
- net a13: now also U1.3 (I3)
- net a14: now also U1.2 (I2)
- net a15: now also U1.1 (I1)
- net a4: now also U1.13 (I13)
- net a5: now also U1.11 (I11)
- net a6: now also U1.10 (I10)
- net a7: now also U1.9 (I9)
- net a8: now also U1.8 (I8)
- net a9: now also U1.7 (I7)
- net phi2: now also U1.23 (I23)
- net r_~w: now also U1.19 (IO19)
- net ~cs_par: now also U1.16 (IO16)
- net ~cs_ser: now also U1.15 (IO15)
- new net: JP1.2 (Pin_2), U1.14 (I14)
- new net cba: U1.21 (IO21)
- new net cst_motor: U1.17 (IO17)
- new net cst_sense_in: U1.18 (IO18)
- new net cst_sense_out: U1.20 (I020)
- new net gab: U1.22 (IO22)
- no-connect marks 21 -> 20
Other:
- note added: "OR GAL22V16"
- moved on the sheet: C1

Commit message: WIP
Parts:
- added U4: 74LS652, Package_DIP:DIP-24_W7.62mm_Socket_LongPads, symbol 74LS652:74LS652
Connections:
- net +5V: now also U4.24 (VCC)
- net GND: now also U4.1 (CAB), U4.12 (GND), U4.2 (SAB)
Changed lines of the file:
@@
 Wire Bus Line
 	5415 1570 4920 1570
+Text Notes 6580 3200 0    50   ~ 0
+OR GAL22V16
+$Comp
+L 74LS652:74LS652 U4
+U 1 1 63CCDE81
+P 9915 4510
+F 0 "U4" H 9915 5425 50  0000 C CNN
+F 1 "74LS652" H 9915 5334 50  0000 C CNN
+F 2 "Package_DIP:DIP-24_W7.62mm_Socket_LongPads" H 9915 4510 50  0001 C CNN
+F 3 "DOCUMENTATION" H 9915 4510 50  0001 C CNN
+	1    9915 4510
+	1    0    0    -1
+$EndComp
+Wire Wire Line
+	9020 3960 9020 4060
+Wire Wire Line
+	9165 3960 9020 3960
+Wire Wire Line
+	9165 4060 9020 4060
+Connection ~ 9020 4060
+Wire Wire Line
+	9020 4060 9020 5060
+$Comp
+L power:GND #PWR0127
+U 1 1 63D05BAE
+P 9020 5375
+F 0 "#PWR0127" H 9020 5125 50  0001 C CNN
+F 1 "GND" H 9025 5202 50  0000 C CNN
+F 2 "" H 9020 5375 50  0001 C CNN
+F 3 "" H 9020 5375 50  0001 C CNN
+	1    9020 5375
+	1    0    0    -1
+$EndComp
+Wire Wire Line
+	10665 3960 10805 3960
+Wire Wire Line
+	10805 3960 10805 3735
+$Comp
+L power:+5V #PWR0128
+U 1 1 63D3BF6E
+P 10805 3735
+F 0 "#PWR0128" H 10805 3585 50  0001 C CNN
+F 1 "+5V" H 10820 3908 50  0000 C CNN
+F 2 "" H 10805 3735 50  0001 C CNN
+F 3 "" H 10805 3735 50  0001 C CNN
+	1    10805 3735
+	1    0    0    -1
+$EndComp
+Wire Wire Line
+	9165 5060 9020 5060
 Wire Bus Line
 	15685 1855 15685 3385
@@
 Wire Bus Line
 	5420 1565 5420 2670
-Text Notes 6580 3200 0    50   ~ 0
-OR GAL22V16
+Connection ~ 9020 5060
+Wire Wire Line
+	9020 5060 9020 5375
 $EndSCHEMATC

Commit message: WIP
Parts:
- added D? (x8): D, symbol Device:D
Connections:
- net +5V: now also U4.22 (SA)
- net GND: now also U4.21 (~G~BA)
- net cba: now also U4.23 (CBA)
- net d0: now also U4.20 (B1)
- net d1: now also U4.19 (B2)
- net d2: now also U4.18 (B3)
- net d3: now also U4.17 (B4)
- net d4: now also U4.16 (B5)
- net d5: now also U4.15 (B6)
- net d6: now also U4.14 (B7)
- net d7: now also U4.13 (B8)
- net gab: now also U4.3 (GAB)
- net p0: now also D?.1 (K)
- net p1: now also D?.1 (K)
- net p2: now also D?.1 (K)
- net p3: now also D?.1 (K)
- net p4: now also D?.1 (K)
- net p5: now also D?.1 (K)
- net p6: now also D?.1 (K)
- net p7: now also D?.1 (K)
- net at U4.10 (A7): now also D?.2 (A)
- net at U4.11 (A8): now also D?.2 (A)
- net at U4.4 (A1): now also D?.2 (A)
- net at U4.5 (A2): now also D?.2 (A)
- net at U4.6 (A3): now also D?.2 (A)
- net at U4.7 (A4): now also D?.2 (A)
- net at U4.8 (A5): now also D?.2 (A)
- net at U4.9 (A6): now also D?.2 (A)
Changed lines of the file:
@@
 Wire Wire Line
 	9165 5060 9020 5060
+Connection ~ 9020 5060
+Wire Wire Line
+	9020 5060 9020 5375
+Wire Wire Line
+	9165 4160 7840 4160
+Wire Wire Line
+	10665 4060 11030 4060
+Text Label 7840 4160 0    50   ~ 0
+gab
+Text Label 11030 4060 2    50   ~ 0
+cba
+Wire Wire Line
+	10805 3960 10805 4160
+Wire Wire Line
+	10805 4160 10665 4160
+Connection ~ 10805 3960
+Wire Wire Line
+	10665 4260 10805 4260
+$Comp
+L power:GND #PWR0129
+U 1 1 63E509B2
+P 10805 5375
+F 0 "#PWR0129" H 10805 5125 50  0001 C CNN
+F 1 "GND" H 10810 5202 50  0000 C CNN
+F 2 "" H 10805 5375 50  0001 C CNN
+F 3 "" H 10805 5375 50  0001 C CNN
+	1    10805 5375
+	1    0    0    -1
+$EndComp
+Wire Wire Line
+	10805 4260 10805 5375
+Wire Wire Line
+	9165 4260 8425 4260
+Wire Wire Line
+	9165 4360 8730 4360
+Wire Wire Line
+	9165 4460 8425 4460
+Wire Wire Line
+	9165 4560 8730 4560
+Wire Wire Line
+	9165 4660 8420 4660
+Wire Wire Line
+	9165 4760 8730 4760
+Wire Wire Line
+	9165 4860 8420 4860
+Wire Wire Line
+	9165 4960 8730 4960
+Entry Wire Line
+	7840 4360 7940 4260
+Entry Wire Line
+	7840 4460 7940 4360
+Entry Wire Line
+	7840 4560 7940 4460
+Entry Wire Line
+	7840 4660 7940 4560
+Entry Wire Line
+	7840 4760 7940 4660
+Entry Wire Line
+	7840 4860 7940 4760
+Entry Wire Line
+	7840 4960 7940 4860
+Entry Wire Line
+	7840 5060 7940 4960
+Wire Bus Line
+	7840 5060 7305 5060
+Text Label 7305 5060 0    50   ~ 0
+parallel_port
+Text Label 7940 4260 0    50   ~ 0
+p0
+Text Label 7940 4360 0    50   ~ 0
+p1
+Text Label 7940 4460 0    50   ~ 0
+p2
+Text Label 7940 4560 0    50   ~ 0
+p3
+Text Label 7940 4660 0    50   ~ 0
+p4
+Text Label 7940 4760 0    50   ~ 0
+p5
+Text Label 7940 4860 0    50   ~ 0
+p6
+Text Label 7940 4960 0    50   ~ 0
+p7
+Wire Wire Line
+	10665 4360 10940 4360
+Wire Wire Line
+	10665 4460 10940 4460
+Wire Wire Line
+	10665 4560 10940 4560
+Wire Wire Line
+	10665 4660 10940 4660
+Wire Wire Line
+	10665 4760 10940 4760
+Wire Wire Line
+	10665 4860 10940 4860
+Wire Wire Line
+	10665 4960 10940 4960
+Wire Wire Line
+	10665 5060 10940 5060
+Entry Wire Line
+	11040 4460 10940 4360
+Entry Wire Line
+	11040 4560 10940 4460
+Entry Wire Line
+	11040 4660 10940 4560
+Entry Wire Line
+	11040 4760 10940 4660
+Entry Wire Line
+	11040 4860 10940 4760
+Entry Wire Line
+	11040 4960 10940 4860
+Entry Wire Line
+	11040 5060 10940 4960
+Entry Wire Line
+	11040 5160 10940 5060
+Wire Bus Line
+	11040 5160 11450 5160
+Text Label 11450 5160 2    50   ~ 0
+data_bus
+Text Label 10940 4360 2    50   ~ 0
+d0
+Text Label 10940 4460 2    50   ~ 0
+d1
+Text Label 10940 4560 2    50   ~ 0
+d2
+Text Label 10940 4660 2    50   ~ 0
+d3
+Text Label 10940 4760 2    50   ~ 0
+d4
+Text Label 10940 4860 2    50   ~ 0
+d5
+Text Label 10940 4960 2    50   ~ 0
+d6
+Text Label 10940 5060 2    50   ~ 0
+d7
 Wire Bus Line
 	15685 1855 15685 3385
@@
 	5680 6205 5680 6905
 Wire Bus Line
+	7840 4360 7840 5060
+Wire Bus Line
+	11040 4460 11040 5160
+Wire Bus Line
 	3630 2205 3630 3705
 Wire Bus Line
 	5420 1565 5420 2670
-Connection ~ 9020 5060
-Wire Wire Line
-	9020 5060 9020 5375
+$Comp
+L Device:D D?
+U 1 1 63ECF378
+P 8275 4260
+F 0 "D?" H 8275 4477 50  0000 C CNN
+F 1 "D" H 8275 4386 50  0000 C CNN
+F 2 "" H 8275 4260 50  0001 C CNN
+F 3 "~" H 8275 4260 50  0001 C CNN
+	1    8275 4260
+	1    0    0    -1
+$EndComp
+Wire Wire Line
+	8125 4260 7940 4260
+$Comp
+L Device:D D?
+U 1 1 63ECFC63
+P 8580 4360
+F 0 "D?" H 8580 4577 50  0000 C CNN
+F 1 "D" H 8580 4486 50  0000 C CNN
+F 2 "" H 8580 4360 50  0001 C CNN
+F 3 "~" H 8580 4360 50  0001 C CNN
+	1    8580 4360
+	1    0    0    -1
+$EndComp
+Wire Wire Line
+	8430 4360 7940 4360
+$Comp
+L Device:D D?
+U 1 1 63ED0FEE
+P 8275 4460
+F 0 "D?" H 8275 4677 50  0000 C CNN
+F 1 "D" H 8275 4586 50  0000 C CNN
+F 2 "" H 8275 4460 50  0001 C CNN
+F 3 "~" H 8275 4460 50  0001 C CNN
+	1    8275 4460
+	1    0    0    -1
+$EndComp
+Wire Wire Line
+	8125 4460 7940 4460
+$Comp
+L Device:D D?
+U 1 1 63ED1611
+P 8270 4660
+F 0 "D?" H 8270 4877 50  0000 C CNN
+F 1 "D" H 8270 4786 50  0000 C CNN
+F 2 "" H 8270 4660 50  0001 C CNN
+F 3 "~" H 8270 4660 50  0001 C CNN
+	1    8270 4660
+	1    0    0    -1
+$EndComp
+Wire Wire Line
+	8120 4660 7940 4660
+$Comp
+L Device:D D?
+U 1 1 63ED1C7A
+P 8270 4860
+F 0 "D?" H 8270 5077 50  0000 C CNN
+F 1 "D" H 8270 4986 50  0000 C CNN
+F 2 "" H 8270 4860 50  0001 C CNN
+F 3 "~" H 8270 4860 50  0001 C CNN
+	1    8270 4860
+	1    0    0    -1
+$EndComp
+Wire Wire Line
+	8120 4860 7940 4860
+$Comp
+L Device:D D?
+U 1 1 63ED2270
+P 8580 4560
+F 0 "D?" H 8580 4777 50  0000 C CNN
+F 1 "D" H 8580 4686 50  0000 C CNN
+F 2 "" H 8580 4560 50  0001 C CNN
+F 3 "~" H 8580 4560 50  0001 C CNN
+	1    8580 4560
+	1    0    0    -1
+$EndComp
+Wire Wire Line
+	8430 4560 7940 4560
+$Comp
+L Device:D D?
+U 1 1 63ED2726
+P 8580 4760
+F 0 "D?" H 8580 4977 50  0000 C CNN
+F 1 "D" H 8580 4886 50  0000 C CNN
+F 2 "" H 8580 4760 50  0001 C CNN
+F 3 "~" H 8580 4760 50  0001 C CNN
+	1    8580 4760
+	1    0    0    -1
+$EndComp
+Wire Wire Line
+	8430 4760 7940 4760
+$Comp
+L Device:D D?
+U 1 1 63ED2E3E
+P 8580 4960
+F 0 "D?" H 8580 5177 50  0000 C CNN
+F 1 "D" H 8580 5086 50  0000 C CNN
+F 2 "" H 8580 4960 50  0001 C CNN
+F 3 "~" H 8580 4960 50  0001 C CNN
+	1    8580 4960
+	1    0    0    -1
+$EndComp
+Wire Wire Line
+	8430 4960 7940 4960
 $EndSCHEMATC
