File: ExtraUserPort.sch (KiCad schematic (older format))
At the start: 38 parts, among them CN1 EXPANSION_PORT, CN2 ALMOST_USERPORT, CN3 DB9_MALE, J1 ATTENTION_IN, J2 TAPE_IN, U1 GAL20V8, U102 74LS652, U2 MOS_6529, U3 MOS_6551_ACIA, U4 MAX238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

Commit message: Final touches
Other:
- note added: "THE IDEA HERE IS TO USE A Y-CABLE AND CONNECT\nTHE DATASSETTE BOTH TO THE ORIGINAL PORT AND TO\nTHIS ONE, SO THAT WE CAN PUT THE SENSE SIGNAL ON\nD2 WHEN REQUIRED.\n\nIDEALLY THE SENSE LINE SHOULD BE BROUGHT HERE\nONLY, BUT PROBABLY IT WON'T HARM ANYWAY.\n\n"
Changed lines of the file:
@@
 Wire Bus Line
 	7140 9770 7140 9775
-Text Notes 6290 9345 0    50   ~ 0
+Text Notes 6275 9430 0    50   ~ 0
 CASSETTE SENSE
 $Comp
@@
 Wire Wire Line
 	5790 9675 6565 9675
+Text Notes 6350 10750 0    50   ~ 0
+THE IDEA HERE IS TO USE A Y-CABLE AND CONNECT\nTHE DATASSETTE BOTH TO THE ORIGINAL PORT AND TO\nTHIS ONE, SO THAT WE CAN PUT THE SENSE SIGNAL ON\nD2 WHEN REQUIRED.\n\nIDEALLY THE SENSE LINE SHOULD BE BROUGHT HERE\nONLY, BUT PROBABLY IT WON'T HARM ANYWAY.\n\n
 Wire Bus Line
 	15640 1415 15640 2945
