File: ExtraUserPort.kicad_pcb (KiCad board)
At the start: 2 copper layers, 60.8 x 99.9 mm, 24 parts, among them CN1 EXPANSION_PORT, CN2 ALMOST_USERPORT, CN3 DB9_MALE, J1 ATTENTION_IN, U1 GAL20V8, U2 MOS_6529, U3 MOS_6551_ACIA, U4 74LS652, U5 MAX238, Y1 1.8432M

Commit message: WIP
Parts:
- added REF**: R_Array_SIP9, Resistor_THT:R_Array_SIP9, F.Cu at (123.8, 125.1)
- moved C3 7.56 mm to (172.8, 93.5), turned to 0 degrees
- moved C7 3.81 mm to (133.8, 84.6)
- moved C9 3.81 mm to (142.1, 84.6)
- moved U4 3.05 mm to (134.6, 130.2)
- moved U2 3.05 mm to (137.8, 125.1)
- moved U3 2.54 mm to (144.9, 112.4)
Connections:
- U1 pad 21: (no net) -> /cba
- U1 pad 22: (no net) -> /gab
- U4 pad 10: (no net) -> /p6
- U4 pad 11: (no net) -> /p7
- U4 pad 13: (no net) -> /d7
- U4 pad 14: (no net) -> /d6
- U4 pad 15: (no net) -> /d5
- U4 pad 16: (no net) -> /d4
- U4 pad 17: (no net) -> /d3
- U4 pad 18: (no net) -> /d2
- U4 pad 19: (no net) -> /d1
- U4 pad 20: (no net) -> /d0
- U4 pad 21: (no net) -> GND
- U4 pad 22: (no net) -> +5V
- U4 pad 23: (no net) -> /cba
- U4 pad 3: (no net) -> /gab
- U4 pad 4: (no net) -> /p0
- U4 pad 5: (no net) -> /p1
- U4 pad 6: (no net) -> /p2
- U4 pad 7: (no net) -> /p3
- U4 pad 8: (no net) -> /p4
- U4 pad 9: (no net) -> /p5
Routing:
- net /a0: track 11.2 -> 39.9 mm, vias 0 -> 1
- net /cba: track 0.00 -> 28.7 mm
- net /a1: track 13.4 -> 39.7 mm, vias 0 -> 1
- net +5V: track 264.0 -> 286.7 mm
- net /p1: track 69.0 -> 48.0 mm, vias 4 -> 3
- net /p0: track 93.1 -> 72.4 mm
- net /gab: track 0.00 -> 17.5 mm
- net /d0: track 95.3 -> 105.8 mm
- net /d1: track 92.0 -> 100.6 mm
- net /d2: track 88.6 -> 95.5 mm
- net /d3: track 85.2 -> 91.3 mm
- net /r_~w: track 70.0 -> 75.8 mm, vias 2 -> 3
- net /rxd_ttl: track 87.5 -> 93.1 mm, vias 3 -> 4
- net /~dsr_ttl: track 74.6 -> 79.4 mm
- net /~cs_par: track 47.8 -> 52.2 mm, vias 1 -> 3
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
Commit message: WIP
Parts:
- added D1: 1n4148, Diode_THT:D_DO-35_SOD27_P2.54mm_Vertical_KathodeUp, F.Cu at (87.3, 106.9)
- added D2: 1n4148, Diode_THT:D_DO-35_SOD27_P2.54mm_Vertical_KathodeUp, F.Cu at (87.3, 110.7)
- added D3: 1n4148, Diode_THT:D_DO-35_SOD27_P2.54mm_Vertical_KathodeUp, F.Cu at (93.3, 106.9)
- added D4: 1n4148, Diode_THT:D_DO-35_SOD27_P2.54mm_Vertical_KathodeUp, F.Cu at (87.3, 114.5)
- added D5: 1n4148, Diode_THT:D_DO-35_SOD27_P2.54mm_Vertical_KathodeUp, F.Cu at (93.3, 110.7)
- added D6: 1n4148, Diode_THT:D_DO-35_SOD27_P2.54mm_Vertical_KathodeUp, F.Cu at (99.3, 106.9)
- added D7: 1n4148, Diode_THT:D_DO-35_SOD27_P2.54mm_Vertical_KathodeUp, F.Cu at (93.3, 114.5)
- added D8: 1n4148, Diode_THT:D_DO-35_SOD27_P2.54mm_Vertical_KathodeUp, F.Cu at (99.3, 110.7)
- RN1: renamed from REF**; value R_Array_SIP9 -> 8.2k
Connections:
- CN2 pad 4: /p2 -> /pc2
- CN2 pad 5: /p3 -> /pc3
- CN2 pad 6: /p4 -> /pc4
- CN2 pad 7: /p5 -> /pc5
- CN2 pad B: /p0 -> /pc0
- CN2 pad F: /p7 -> /pc7
- CN2 pad J: /p6 -> /pc6
- CN2 pad K: /p1 -> /pc1
- RN1 pad 1: (no net) -> +5V
- RN1 pad 2: (no net) -> /pc0
- RN1 pad 3: (no net) -> /pc1
- RN1 pad 4: (no net) -> /pc2
- RN1 pad 5: (no net) -> /pc3
- RN1 pad 6: (no net) -> /pc4
- RN1 pad 7: (no net) -> /pc5
- RN1 pad 8: (no net) -> /pc6
- RN1 pad 9: (no net) -> /pc7
- U1 pad 22: /gab -> (no net)
- U4 pad 3: /gab -> (no net)
Routing:
- net /pc2: track 0.00 -> 88.6 mm, vias 0 -> 2
- net /p2: track 91.8 -> 3.17 mm, vias 2 -> 0
- net /pc3: track 0.00 -> 76.7 mm, vias 0 -> 2
- net /p3: track 79.9 -> 3.17 mm, vias 2 -> 0
- net /pc4: track 0.00 -> 70.5 mm, vias 0 -> 2
- net /p4: track 74.8 -> 4.32 mm, vias 2 -> 0
- net /pc0: track 0.00 -> 69.2 mm, vias 0 -> 3
- net /p0: track 72.4 -> 3.17 mm, vias 3 -> 0
- net +5V: track 286.7 -> 232.1 mm
- net /pc1: track 0.00 -> 44.8 mm, vias 0 -> 3
- net /p1: track 48.0 -> 3.17 mm, vias 3 -> 0
- net /gab: track 17.5 -> 0.00 mm
- net (no net): track 0.00 -> 17.5 mm
- net /p5: track 74.8 -> 64.4 mm
- net /p7: track 69.1 -> 63.9 mm
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
Commit message: WIP
Parts:
- added REF**: Connector_Mini-DIN_Female_8Pin_2rows, ExtraUserPort:Connector_Mini-DIN_Female_8Pin_2rows, F.Cu at (129.9, 93.1)
- D1, D2, D3, D4, D5, D6, D7, D8: value 1n4148 -> BAT43
- R1, R2, R3: footprint Resistor_THT:R_Axial_DIN0207_L6.3mm_D2.5mm_P10.16mm_Horizontal -> Resistor_THT:R_Axial_DIN0207_L6.3mm_D2.5mm_P2.54mm_Vertical
- moved D7 63.5 mm to (151.3, 88.5)
- moved D6 56.5 mm to (151.3, 84.7)
- moved D2 55.5 mm to (128.5, 73.5), turned to 180 degrees
- moved D8 55.1 mm to (151.3, 92.3)
- moved D1 54.7 mm to (128.5, 71.0), turned to 180 degrees
- moved D4 54.6 mm to (128.5, 78.6), turned to 180 degrees
- moved D3 46.8 mm to (128.5, 76.1), turned to 180 degrees
- moved D5 45.9 mm to (128.5, 81.2), turned to 180 degrees
- moved RN1 16.6 mm to (116.3, 110.2)
- moved R1 7.62 mm to (157.6, 84.7)
- moved R2 7.62 mm to (157.6, 88.5)
- moved R3 7.62 mm to (157.6, 92.3)
- moved C7 3.81 mm to (137.6, 84.6)
- moved C9 1.90 mm to (144.0, 84.6), turned to 0 degrees
Connections:
- D1 pad 1: /pc0 -> /p0
- D1 pad 2: /p0 -> /pc0
- D2 pad 1: /pc1 -> /p1
- D2 pad 2: /p1 -> /pc1
- D3 pad 1: /pc2 -> /p2
- D3 pad 2: /p2 -> /pc2
- D4 pad 1: /pc3 -> /p3
- D4 pad 2: /p3 -> /pc3
- D5 pad 1: /pc4 -> /p4
- D5 pad 2: /p4 -> /pc4
- D6 pad 1: /pc5 -> /p5
- D6 pad 2: /p5 -> /pc5
- D7 pad 1: /pc6 -> /p6
- D7 pad 2: /p6 -> /pc6
- D8 pad 1: /pc7 -> /p7
- D8 pad 2: /p7 -> /pc7
- U1 pad 22: (no net) -> /gab
- U4 pad 3: (no net) -> /gab
Routing:
- net /p0: track 3.17 -> 62.1 mm
- net /p1: track 3.17 -> 56.5 mm
- net /p2: track 3.17 -> 50.8 mm
- net /pc5: track 0.00 -> 46.8 mm, vias 0 -> 2
- net /pc6: track 0.00 -> 44.8 mm, vias 0 -> 1
- net /pc7: track 0.00 -> 44.4 mm, vias 0 -> 1
- net /pc2: track 88.6 -> 47.6 mm
- net /pc3: track 76.7 -> 37.1 mm
- net /pc4: track 70.5 -> 32.1 mm
- net /p3: track 3.17 -> 41.1 mm
- net /p7: track 63.9 -> 26.0 mm, vias 2 -> 1
- net /p6: track 62.2 -> 30.2 mm, vias 2 -> 1
- net /p5: track 64.4 -> 35.3 mm, vias 3 -> 1
- net /pc1: track 44.8 -> 24.6 mm
- net /pc0: track 69.2 -> 49.1 mm
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
Commit message: WIP
Parts:
- removed REF**: Connector_Mini-DIN_Female_8Pin_2rows, ExtraUserPort:Connector_Mini-DIN_Female_8Pin_2rows
- moved RN1 30.1 mm to (124.3, 81.2)
- moved C5 5.08 mm to (145.2, 67.3)
- moved C6 5.08 mm to (140.8, 67.3)
- moved U5 5.08 mm to (165.2, 72.1)
- moved C8 5.08 mm to (153.5, 67.3)
- moved C9 3.18 mm to (147.1, 84.6), turned to 180 degrees
- moved J1 2.92 mm to (130.2, 67.3)
- moved D1 1.68 mm to (130.2, 71.0), turned to 0 degrees
- moved D2 1.68 mm to (130.2, 73.5), turned to 0 degrees
- moved D3 1.68 mm to (130.2, 76.1), turned to 0 degrees
- moved D4 1.68 mm to (130.2, 78.6), turned to 0 degrees
- moved D5 1.68 mm to (130.2, 81.2), turned to 0 degrees
- moved C7 1.27 mm to (138.9, 84.6)
Connections:
- RN1 pad 2: /pc0 -> /pc4
- RN1 pad 3: /pc1 -> /pc3
- RN1 pad 5: /pc3 -> /pc1
- RN1 pad 6: /pc4 -> /pc0
Routing:
- net +5V: track 224.5 -> 285.0 mm, vias 3 -> 2
- net /pc4: track 32.1 -> 63.8 mm
- net /pc7: track 44.4 -> 73.3 mm, vias 1 -> 2
- net /pc3: track 37.1 -> 65.0 mm
- net /pc2: track 47.6 -> 72.1 mm
- net /pc1: track 24.6 -> 47.4 mm
- net /pc0: track 49.1 -> 69.0 mm
- net /pc6: track 44.8 -> 64.6 mm, vias 1 -> 2
- net /pc5: track 46.8 -> 65.7 mm
- net /p4: track 21.4 -> 38.9 mm
- net /rxc_ttl: track 78.4 -> 88.0 mm
- net /~dsr_ttl: track 79.4 -> 87.0 mm
- net /~dsr: track 20.5 -> 15.4 mm
- net /~dtr: track 29.9 -> 24.9 mm
- net /rxd: track 32.6 -> 27.5 mm
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
Commit message: WIP
Parts:
- added J2: TAPE_IN, ExtraUserPort:Connector_Mini-DIN_Female_8Pin_2rows, F.Cu at (129.8, 93.1)
- added JP4: JMP_CASS_SENSE, Jumper:SolderJumper-2_P1.3mm_Bridged_RoundedPad1.0x1.5mm, B.Cu at (135.6, 90.2)
Routing:
- net /pc2: track 72.1 -> 86.7 mm, vias 2 -> 3
- net /~cassette_sense: track 0.00 -> 2.92 mm
- net /p3: track 45.6 -> 44.5 mm
- net /~rts_ttl: track 93.6 -> 92.7 mm

Commit message: WIP
Parts:
- moved C2 13.0 mm to (123.7, 125.1), turned to 90 degrees
- moved Y1 2.54 mm to (162.6, 117.5)
- moved JP1 1.52 mm to (177.9, 128.9)
- moved C1 0.13 mm to (141.0, 123.8)
- renumbered U4 to U102, U5 to U4
Routing:
- net /~cs_par: track 51.6 -> 37.5 mm, vias 3 -> 0
- net +5V: track 285.0 -> 297.1 mm, vias 2 -> 3
- net /phi2: track 77.4 -> 71.6 mm
- net /d7: track 77.3 -> 81.5 mm
- net /d4: track 88.7 -> 92.9 mm
- net /d3: track 91.1 -> 95.3 mm
- net /d5: track 84.0 -> 88.2 mm
- net /d2: track 95.4 -> 99.6 mm
- net /d6: track 80.7 -> 84.9 mm
- net /a1: track 39.7 -> 43.7 mm, vias 1 -> 2
- net /~cs_ser: track 27.5 -> 31.1 mm
- net /d0: track 105.6 -> 109.0 mm
- net /d1: track 100.4 -> 103.8 mm
- net Net-(U3-Pad6): track 7.73 -> 5.13 mm, vias 1 -> 0
- net /r_~w: track 75.0 -> 76.8 mm
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Other:
- board text added: "GAL20V8 or GAL22V16"
- board text added: "↑6529 ↓74652"
- board text removed: "MOS 6529"

Commit message: WIP
Parts:
- moved D6 2.54 mm to (153.8, 84.7)
- moved D7 2.54 mm to (153.8, 88.5)
- moved D8 2.54 mm to (153.8, 92.3)
- moved JP2 2.54 mm to (143.6, 90.7)
- moved JP3 2.54 mm to (143.6, 93.2)
- moved R1 2.54 mm to (160.1, 84.7)
- moved R2 2.54 mm to (160.1, 88.5)
- moved R3 2.54 mm to (160.1, 92.3)
Routing:
- net Net-(JP3-Pad2): track 45.3 -> 41.4 mm, vias 2 -> 1
- net /p5: track 35.3 -> 38.1 mm
- net /pc6: track 64.6 -> 67.3 mm
- net /~dsr_ttl: track 87.0 -> 84.4 mm
- net /~dcd_ttl: track 79.8 -> 77.2 mm
- net /~rts: track 16.0 -> 14.2 mm
- net /p6: track 30.2 -> 31.6 mm
- net Net-(JP2-Pad2): track 35.7 -> 36.8 mm
- net /pc7: track 73.3 -> 72.2 mm
- net /pc5: track 65.7 -> 64.7 mm
- net /p7: track 26.0 -> 27.1 mm
- net /~dsr: track 15.4 -> 14.7 mm
- net /~dtr_ttl: track 79.5 -> 80.0 mm, vias 5 -> 6

Commit message: WIP
Routing:
- net /~dcd_ttl: track 77.2 -> 96.2 mm, vias 3 -> 5
- net /pc2: track 86.7 -> 90.1 mm
- net +5V: track 297.1 -> 300.0 mm
- net /pc6: track 67.3 -> 64.9 mm
- net /d4: track 92.9 -> 91.6 mm
- net /~dsr_ttl: track 84.4 -> 83.3 mm
- net /pc5: track 64.7 -> 63.6 mm, vias 2 -> 1
- net /pc4: track 63.8 -> 62.8 mm
- net /~irq: track 55.8 -> 54.9 mm
- net /pc7: track 72.2 -> 73.0 mm
- net GND: vias 10 -> 11
