File: 16up.kicad_pcb (KiCad board)
At the start: 2 copper layers, 60.8 x 99.9 mm, 20 parts, among them CN1 EXPANSION_PORT, CN2 ALMOST_USERPORT, CN4 TAPE_IN, J1 ATTENTION_IN, U1 GAL20V8, U102 74LS652, U2 MOS_6529, U3 MOS_6551_ACIA, U4 74HCT04, Y1 1.8432M

Commit message: WIP
Parts:
- moved CN2 16.3 mm to (152.2, 74.0)
Routing:
- net /txd_ttl: track 96.8 -> 46.8 mm
- net /dsr_ttl: track 89.5 -> 73.5 mm
- net /rxd_ttl: track 85.5 -> 69.6 mm
- net /dcd_ttl: track 81.4 -> 65.7 mm
- net /~reset: track 113.6 -> 97.9 mm
- net /dtr_ttl: track 38.9 -> 25.7 mm
- net +5V: track 225.7 -> 213.4 mm
- net /rts_ttl: track 28.9 -> 17.2 mm
- net /rxc: track 68.0 -> 61.0 mm
- net /p2: track 112.1 -> 109.3 mm
- net /p7: track 86.9 -> 84.2 mm
- net /p0: track 114.9 -> 112.3 mm
- net /p3: track 97.6 -> 95.3 mm
- net /p4: track 91.8 -> 90.2 mm
- net /p5: track 86.5 -> 85.2 mm
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Other:
- board size 60.8 x 99.9 mm -> 60.8 x 83.7 mm

Commit message: Almost there
Routing:
- net /txd_ttl: track 46.8 -> 80.9 mm
- net /p4: track 90.2 -> 73.7 mm
- net /p1: track 86.4 -> 69.9 mm
- net /p7: track 84.2 -> 68.0 mm
- net /p5: track 85.2 -> 68.9 mm
- net /p3: track 95.3 -> 79.0 mm
- net /p2: track 109.3 -> 93.1 mm
- net /p0: track 112.3 -> 96.0 mm
- net /p6: track 78.3 -> 62.5 mm
- net /dcd_ttl: track 65.7 -> 53.2 mm, vias 4 -> 3
- net /rxc: track 61.0 -> 51.8 mm
- net /dsr_ttl: track 73.5 -> 77.0 mm
- net /~cs_ser: track 25.9 -> 23.4 mm
- net /~reset: track 97.9 -> 96.3 mm
- net /rxd_ttl: track 69.6 -> 68.7 mm
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Other:
- board text added: "DCD"
- board text added: "DSR"
- board text added: "DTR"
- board text added: "RTS"
- board text added: "RXC"
- board text added: "RXD"
- board text added: "TXD"

Commit message: Routing done
Parts:
- removed J1: ATTENTION_IN, Connector_PinHeader_2.54mm:PinHeader_1x01_P2.54mm_Vertical
- added J3: CONN_UPORT254, Connector_PinHeader_2.54mm:PinHeader_2x12_P2.54mm_Vertical, F.Cu at (155.7, 77.9)
- moved R2 25.7 mm to (177.9, 76.3), turned to 180 degrees
- moved R1 18.2 mm to (172.8, 76.3), turned to 180 degrees
- moved CN2 1.27 mm to (152.2, 72.7)
Connections:
- CN2 pad 10: Net-(CN2-Pad10) -> /+9v
- CN2 pad 11: Net-(CN2-Pad11) -> /-9v
- CN2 pad 9: Net-(CN2-Pad9) -> /~attn
Routing:
- net /rts_ttl: track 17.2 -> 45.1 mm, vias 1 -> 0
- net /rxd_ttl: track 68.7 -> 96.0 mm, vias 2 -> 3
- net /dtr_ttl: track 25.7 -> 49.3 mm, vias 2 -> 0
- net /~reset: track 96.3 -> 115.8 mm, vias 3 -> 6
- net /p1: track 69.9 -> 88.3 mm, vias 3 -> 2
- net /dcd_ttl: track 53.2 -> 70.3 mm, vias 3 -> 1
- net /~attn: track 0.00 -> 16.0 mm
- net /rxc: track 51.8 -> 67.5 mm, vias 1 -> 3
- net /+9v: track 0.00 -> 14.7 mm
- net /-9v: track 0.00 -> 14.1 mm
- net Net-(CN2-Pad9): track 7.58 -> 0.00 mm
- net /p0: track 96.0 -> 90.1 mm, vias 3 -> 0
- net /txd_ttl: track 80.9 -> 86.6 mm, vias 3 -> 1
- net /p2: track 93.1 -> 88.5 mm, vias 3 -> 1
- net /r_~w: track 119.5 -> 123.7 mm
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Other:
- board size 60.8 x 83.7 mm -> 60.8 x 85 mm
- net class NineVolts added: clearance 0.1, trace_width 0.5, via_dia 0.8, via_drill 0.6
- board text added: "+9VAC"
- board text added: "-9VAC"
- board text added: "NOTES: - ON PLUS/4 USE EXTERNAL ADDRESS ONLY (ACIA = $FD6x, 6529 = $FD7x) - ON C16 INTERNAL ADDRESS REQUIRES MODIFICATION (ACIA = $FD0x, 6529 = $FD1x) - DO NOT MOUNT RN1 IF USING ORIGINAL MOS 6529 - IF NEEDED, ~ATTN~ AND ±9V MUST BE PROVIDED EXTERNALLY THROUGH J3"
- board text removed: "NOTES: - ON PLUS/4 USE EXTERNAL ADDRESS ONLY (ACIA = $FD6x, 6529 = $FD7x) - ON C16 INTERNAL ADDRESS REQUIRES MODIFICATION (ACIA = $FD0x, 6529 = $FD1x) - DO NOT MOUNT RN1 IF USING ORIGINAL MOS 6529"
- board text removed: "~ATTN IN"

Commit message: Final touches
Routing:
- net /txd_ttl: track 86.6 -> 88.6 mm
- net /dcd_ttl: track 70.3 -> 71.2 mm
- net GND: vias 6 -> 9
Other:
- board text added: "NOTES: - ON PLUS/4 USE EXTERNAL ADDRESS ONLY (ACIA = $FD6x, 6529 = $FD7x) - ON C16 INTERNAL ADDRESS REQUIRES MODIFICATION (ACIA = $FD0x, 6529 = $FD1x) - DO NOT MOUNT RN1 IF USING ORIGINAL MOS 6529 - IF REQUIRED, ~ATTN~ AND ±9V MUST BE PROVIDED EXTERNALLY THROUGH J3"
- board text removed: "NOTES: - ON PLUS/4 USE EXTERNAL ADDRESS ONLY (ACIA = $FD6x, 6529 = $FD7x) - ON C16 INTERNAL ADDRESS REQUIRES MODIFICATION (ACIA = $FD0x, 6529 = $FD1x) - DO NOT MOUNT RN1 IF USING ORIGINAL MOS 6529 - IF NEEDED, ~ATTN~ AND ±9V MUST BE PROVIDED EXTERNALLY THROUGH J3"
